Commit message: refactor: changing architecture

File: ros_ws/src/krsti_description/urdf/krsti.xacro (robot description, xacro)
@@ -3,4 +3,26 @@
 <xacro:include filename="$(find krsti_description)/urdf/materials.xacro" />
 <xacro:include filename="$(find krsti_description)/urdf/krsti.trans" />
+<!-- ─── ros2_control ──────────────────────────────────────────────────────── -->
+<ros2_control name="GazeboSystem" type="system">
+  <hardware>
+    <plugin>gz_ros2_control/GazeboSimSystem</plugin>
+  </hardware>
+  <joint name="Revolute 5">
+    <command_interface name="position"/>
+    <state_interface name="position"/>
+    <state_interface name="velocity"/>
+  </joint>
+  <joint name="Revolute 6">
+    <command_interface name="position"/>
+    <state_interface name="position"/>
+    <state_interface name="velocity"/>
+  </joint>
+</ros2_control>
+<!-- ─── Gazebo ros2_control plugin ──────────────────────────────────────── -->
+<gazebo>
+  <plugin filename="gz_ros2_control-system" name="gz_ros2_control::GazeboSimROS2ControlPlugin">
+    <parameters>$(find krsti_description)/config/ros2_control.yaml</parameters>
+  </plugin>
+</gazebo>
 <link name="base_link">
   <inertial>
